File: ProMicro_LIPO.sch (KiCad schematic (older format))
At the start: 25 parts, among them J1 JST, U1 MCP73831-2-OT, U2 TPS61090

Commit message: trigger CI run
Changed lines of the file:
@@
 Text Notes 10500 2875 0    50   ~ 0
 TCK
-Text Notes 4000 7250 0    50   ~ 0
+Text Notes 3750 7250 0    50   ~ 0
 close 1-2 read analog voltage\nclose 2-3 read LBO status\nopen 1 2 3 if no battery status required
 $EndSCHEMATC

Commit message: changed SPI signal names
Other:
- note added: "BTN"
- note added: "CS1"
- note added: "RXD"
- note added: "SCK"
- note added: "SDI"
- note added: "SDO"
- note added: "TXD"
- note removed: "CLK"
- note removed: "MISO"
- note removed: "MOSI"
- note removed: "RxD"
- note removed: "TxD"
Changed lines of the file:
@@
 NoConn ~ 10275 1950
 Text Notes 8825 1975 2    50   ~ 0
-RxD
+RXD
 Text Notes 8825 2075 2    50   ~ 0
-TxD
+TXD
 Text Notes 8825 2175 2    50   ~ 0
 SDA
@@
 SCL
 Text Notes 8825 3275 2    50   ~ 0
-CLK
+SCK
 Text Notes 8825 3175 2    50   ~ 0
-MISO
+SDI
 Text Notes 8825 3075 2    50   ~ 0
-MOSI
+SDO
 Text Notes 8825 2975 2    50   ~ 0
 CS0
@@
 	1    0    0    -1
 $EndComp
-Text Notes 8825 2675 2    50   ~ 0
+Text Notes 8825 2775 2    50   ~ 0
 INT0
 Text Notes 10500 2575 0    50   ~ 0
@@
 Text Notes 3750 7250 0    50   ~ 0
 close 1-2 read analog voltage\nclose 2-3 read LBO status\nopen 1 2 3 if no battery status required
+Text Notes 8825 2875 2    50   ~ 0
+CS1
+Text Notes 8825 2575 2    50   ~ 0
+BTN
 $EndSCHEMATC
