File: _TEMPLATE/ProMicro_TEST.kicad_pcb (KiCad board)
At the start: 2 copper layers, 17.8 x 30.5 mm, 6 parts

Commit message: clean
Changed lines of the file:
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@@
-(kicad_pcb (version 20171130) (host pcbnew 5.1.5)
+(kicad_pcb (version 20171130) (host pcbnew 5.1.5+dfsg1-2build2)
   (general
     (thickness 0.8)
@@
       (effects (font (size 1 1) (thickness 0.15)))
     )
-    (pad 1 thru_hole rect (at 0 0 180) (size 1.6 1.6) (drill 0.8) (layers *.Cu *.Mask))
-    (pad 2 thru_hole oval (at 0 2.54 180) (size 1.6 1.6) (drill 0.8) (layers *.Cu *.Mask))
-    (pad 3 thru_hole oval (at 0 5.08 180) (size 1.6 1.6) (drill 0.8) (layers *.Cu *.Mask)
+    (pad 1 thru_hole rect (at 0 0 180) (size 2 2) (drill 1) (layers *.Cu *.Mask))
+    (pad 2 thru_hole oval (at 0 2.54 180) (size 2 2) (drill 1) (layers *.Cu *.Mask))
+    (pad 3 thru_hole oval (at 0 5.08 180) (size 2 2) (drill 1) (layers *.Cu *.Mask)
       (net 1 GND))
-    (pad 13 thru_hole oval (at 15.24 27.94 180) (size 1.6 1.6) (drill 0.8) (layers *.Cu *.Mask))
-    (pad 4 thru_hole oval (at 0 7.62 180) (size 1.6 1.6) (drill 0.8) (layers *.Cu *.Mask)
+    (pad 13 thru_hole oval (at 15.24 27.94 180) (size 2 2) (drill 1) (layers *.Cu *.Mask))
+    (pad 4 thru_hole oval (at 0 7.62 180) (size 2 2) (drill 1) (layers *.Cu *.Mask)
       (net 1 GND))
-    (pad 14 thru_hole oval (at 15.24 25.4 180) (size 1.6 1.6) (drill 0.8) (layers *.Cu *.Mask))
-    (pad 5 thru_hole oval (at 0 10.16 180) (size 1.6 1.6) (drill 0.8) (layers *.Cu *.Mask)
+    (pad 14 thru_hole oval (at 15.24 25.4 180) (size 2 2) (drill 1) (layers *.Cu *.Mask))
+    (pad 5 thru_hole oval (at 0 10.16 180) (size 2 2) (drill 1) (layers *.Cu *.Mask)
       (net 4 SDA))
-    (pad 15 thru_hole oval (at 15.24 22.86 180) (size 1.6 1.6) (drill 0.8) (layers *.Cu *.Mask))
-    (pad 6 thru_hole oval (at 0 12.7 180) (size 1.6 1.6) (drill 0.8) (layers *.Cu *.Mask)
+    (pad 15 thru_hole oval (at 15.24 22.86 180) (size 2 2) (drill 1) (layers *.Cu *.Mask))
+    (pad 6 thru_hole oval (at 0 12.7 180) (size 2 2) (drill 1) (layers *.Cu *.Mask)
       (net 3 SCL))
-    (pad 16 thru_hole oval (at 15.24 20.32 180) (size 1.6 1.6) (drill 0.8) (layers *.Cu *.Mask))
-    (pad 7 thru_hole oval (at 0 15.24 180) (size 1.6 1.6) (drill 0.8) (layers *.Cu *.Mask))
-    (pad 17 thru_hole oval (at 15.24 17.78 180) (size 1.6 1.6) (drill 0.8) (layers *.Cu *.Mask))
-    (pad 8 thru_hole oval (at 0 17.78 180) (size 1.6 1.6) (drill 0.8) (layers *.Cu *.Mask))
-    (pad 18 thru_hole oval (at 15.24 15.24 180) (size 1.6 1.6) (drill 0.8) (layers *.Cu *.Mask))
-    (pad 9 thru_hole oval (at 0 20.32 180) (size 1.6 1.6) (drill 0.8) (layers *.Cu *.Mask))
-    (pad 19 thru_hole oval (at 15.24 12.7 180) (size 1.6 1.6) (drill 0.8) (layers *.Cu *.Mask))
-    (pad 10 thru_hole oval (at 0 22.86 180) (size 1.6 1.6) (drill 0.8) (layers *.Cu *.Mask))
-    (pad 20 thru_hole oval (at 15.24 10.16 180) (size 1.6 1.6) (drill 0.8) (layers *.Cu *.Mask))
-    (pad 11 thru_hole oval (at 0 25.4 180) (size 1.6 1.6) (drill 0.8) (layers *.Cu *.Mask))
-    (pad 21 thru_hole oval (at 15.24 7.62 180) (size 1.6 1.6) (drill 0.8) (layers *.Cu *.Mask)
+    (pad 16 thru_hole oval (at 15.24 20.32 180) (size 2 2) (drill 1) (layers *.Cu *.Mask))
+    (pad 7 thru_hole oval (at 0 15.24 180) (size 2 2) (drill 1) (layers *.Cu *.Mask))
+    (pad 17 thru_hole oval (at 15.24 17.78 180) (size 2 2) (drill 1) (layers *.Cu *.Mask))
+    (pad 8 thru_hole oval (at 0 17.78 180) (size 2 2) (drill 1) (layers *.Cu *.Mask))
+    (pad 18 thru_hole oval (at 15.24 15.24 180) (size 2 2) (drill 1) (layers *.Cu *.Mask))
+    (pad 9 thru_hole oval (at 0 20.32 180) (size 2 2) (drill 1) (layers *.Cu *.Mask))
+    (pad 19 thru_hole oval (at 15.24 12.7 180) (size 2 2) (drill 1) (layers *.Cu *.Mask))
+    (pad 10 thru_hole oval (at 0 22.86 180) (size 2 2) (drill 1) (layers *.Cu *.Mask))
+    (pad 20 thru_hole oval (at 15.24 10.16 180) (size 2 2) (drill 1) (layers *.Cu *.Mask))
+    (pad 11 thru_hole oval (at 0 25.4 180) (size 2 2) (drill 1) (layers *.Cu *.Mask))
+    (pad 21 thru_hole oval (at 15.24 7.62 180) (size 2 2) (drill 1) (layers *.Cu *.Mask)
       (net 2 +3V3))
-    (pad 12 thru_hole oval (at 0 27.94 180) (size 1.6 1.6) (drill 0.8) (layers *.Cu *.Mask))
-    (pad 22 thru_hole oval (at 15.24 5.08 180) (size 1.6 1.6) (drill 0.8) (layers *.Cu *.Mask))
-    (pad 23 thru_hole oval (at 15.24 2.54 180) (size 1.6 1.6) (drill 0.8) (layers *.Cu *.Mask)
+    (pad 12 thru_hole oval (at 0 27.94 180) (size 2 2) (drill 1) (layers *.Cu *.Mask))
+    (pad 22 thru_hole oval (at 15.24 5.08 180) (size 2 2) (drill 1) (layers *.Cu *.Mask))
+    (pad 23 thru_hole oval (at 15.24 2.54 180) (size 2 2) (drill 1) (layers *.Cu *.Mask)
       (net 1 GND))
-    (pad 24 thru_hole oval (at 15.24 0 180) (size 1.6 1.6) (drill 0.8) (layers *.Cu *.Mask))
+    (pad 24 thru_hole oval (at 15.24 0 180) (size 2 2) (drill 1) (layers *.Cu *.Mask))
     (model ${KISYS3DMOD}/Module.3dshapes/Sparkfun_Pro_Micro.wrl
       (at (xyz 0 0 0))
