File: TEST/ProMicro_TEST.sch (KiCad schematic (older format))
At the start: 6 parts

Commit message: update schematic and PCBs
Parts:
- R3, R4: MPN (none) -> RC0402FR-074K7L; manf# RC0402FR-074K7L -> (none)
Changed lines of the file:
@@
 F 2 "Resistor_SMD:R_0402_1005Metric" V 8930 5500 50  0001 C CNN
 F 3 "~" H 9000 5500 50  0001 C CNN
-F 4 "RC0402FR-074K7L" H 9000 5500 50  0001 C CNN "manf#"
+F 4 "RC0402FR-074K7L" H 9000 5500 50  0001 C CNN "MPN"
 	1    9000 5500
 	-1   0    0    1
@@
 F 2 "Resistor_SMD:R_0402_1005Metric" V 9430 5500 50  0001 C CNN
 F 3 "~" H 9500 5500 50  0001 C CNN
-F 4 "RC0402FR-074K7L" H 9500 5500 50  0001 C CNN "manf#"
+F 4 "RC0402FR-074K7L" H 9500 5500 50  0001 C CNN "MPN"
 F 5 "C105871" H 9500 5500 50  0001 C CNN "lcsc#"
 	1    9500 5500
