File: BUS/ProMicro_BUS.kicad_pcb (KiCad board)
At the start: 2 copper layers, 17.8 x 30.5 mm, 15 parts, among them J1 Conn_01x03, U1 MAX3483, U2 MAX3051, U3 MCP2515-xSO, Y1 Crystal

Commit message: update PCBs to be stackable
Parts:
- moved LOGO1 0.64 mm to (59.1, 99.7)
Connections:
- A1 pad 11: (no net) -> Net-(A1-Pad11)
- A1 pad 17: (no net) -> Net-(A1-Pad17)
- A1 pad 18: (no net) -> Net-(A1-Pad18)
- A1 pad 19: (no net) -> Net-(A1-Pad19)
- A1 pad 20: (no net) -> Net-(A1-Pad20)
- A1 pad 24: (no net) -> Net-(A1-Pad24)
- A1 pad 5: (no net) -> Net-(A1-Pad5)
- A1 pad 6: (no net) -> Net-(A1-Pad6)
- A1 pad 7: (no net) -> Net-(A1-Pad7)
- A1 pad 8: (no net) -> Net-(A1-Pad8)
- A1 pad 9: (no net) -> Net-(A1-Pad9)
- U2 pad 5: (no net) -> Net-(U2-Pad5)
- U3 pad 10: (no net) -> Net-(U3-Pad10)
- U3 pad 11: (no net) -> Net-(U3-Pad11)
- U3 pad 3: (no net) -> Net-(U3-Pad3)
- U3 pad 4: (no net) -> Net-(U3-Pad4)
- U3 pad 5: (no net) -> Net-(U3-Pad5)
- U3 pad 6: (no net) -> Net-(U3-Pad6)
Other:
- board text added: "nerdyscout.github.io/ ProMicro/BUS v1.4"
- board text removed: "nerdyscout.github.io/ ProMicro/BUS v1.3"
Changed lines of the file:
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@@
     (zones 0)
     (modules 15)
-    (nets 21)
+    (nets 39)
   )
   (page A4)
@@
   )
   (layers
-    (0 F.Cu mixed)
-    (31 B.Cu mixed)
+    (0 F.Cu mixed hide)
+    (31 B.Cu mixed hide)
     (32 B.Adhes user)
     (33 F.Adhes user)
@@
   (net 19 "Net-(C4-Pad1)")
   (net 20 CS)
+  (net 21 "Net-(A1-Pad5)")
+  (net 22 "Net-(A1-Pad6)")
+  (net 23 "Net-(A1-Pad7)")
+  (net 24 "Net-(A1-Pad17)")
+  (net 25 "Net-(A1-Pad8)")
+  (net 26 "Net-(A1-Pad18)")
+  (net 27 "Net-(A1-Pad9)")
+  (net 28 "Net-(A1-Pad19)")
+  (net 29 "Net-(A1-Pad20)")
+  (net 30 "Net-(A1-Pad11)")
+  (net 31 "Net-(A1-Pad24)")
+  (net 32 "Net-(U2-Pad5)")
+  (net 33 "Net-(U3-Pad11)")
+  (net 34 "Net-(U3-Pad10)")
+  (net 35 "Net-(U3-Pad6)")
+  (net 36 "Net-(U3-Pad5)")
+  (net 37 "Net-(U3-Pad4)")
+  (net 38 "Net-(U3-Pad3)")
   (net_class Default "This is the default net class."
     (clearance 0.2)
@@
     (add_net CS1)
     (add_net INT)
+    (add_net "Net-(A1-Pad11)")
+    (add_net "Net-(A1-Pad17)")
+    (add_net "Net-(A1-Pad18)")
+    (add_net "Net-(A1-Pad19)")
+    (add_net "Net-(A1-Pad20)")
+    (add_net "Net-(A1-Pad24)")
+    (add_net "Net-(A1-Pad5)")
+    (add_net "Net-(A1-Pad6)")
+    (add_net "Net-(A1-Pad7)")
+    (add_net "Net-(A1-Pad8)")
+    (add_net "Net-(A1-Pad9)")
     (add_net "Net-(C1-Pad2)")
     (add_net "Net-(C4-Pad1)")
@@
     (add_net "Net-(U2-Pad1)")
     (add_net "Net-(U2-Pad4)")
+    (add_net "Net-(U2-Pad5)")
+    (add_net "Net-(U3-Pad10)")
+    (add_net "Net-(U3-Pad11)")
+    (add_net "Net-(U3-Pad3)")
+    (add_net "Net-(U3-Pad4)")
+    (add_net "Net-(U3-Pad5)")
+    (add_net "Net-(U3-Pad6)")
     (add_net RXD)
     (add_net SCK)
@@
     (pad 14 thru_hole circle (at 15.24 25.4) (size 2.1 2.1) (drill 1.4) (layers *.Cu *.Mask)
       (net 13 COPI))
-    (pad 5 thru_hole circle (at 0 10.16) (size 2.1 2.1) (drill 1.4) (layers *.Cu *.Mask))
+    (pad 5 thru_hole circle (at 0 10.16) (size 2.1 2.1) (drill 1.4) (layers *.Cu *.Mask)
+      (net 21 "Net-(A1-Pad5)"))
     (pad 15 thru_hole circle (at 15.24 22.86) (size 2.1 2.1) (drill 1.4) (layers *.Cu *.Mask)
       (net 14 CIPO))
-    (pad 6 thru_hole circle (at 0 12.7) (size 2.1 2.1) (drill 1.4) (layers *.Cu *.Mask))
+    (pad 6 thru_hole circle (at 0 12.7) (size 2.1 2.1) (drill 1.4) (layers *.Cu *.Mask)
+      (net 22 "Net-(A1-Pad6)"))
     (pad 16 thru_hole circle (at 15.24 20.32) (size 2.1 2.1) (drill 1.4) (layers *.Cu *.Mask)
       (net 15 SCK))
-    (pad 7 thru_hole circle (at 0 15.24) (size 2.1 2.1) (drill 1.4) (layers *.Cu *.Mask))
-    (pad 17 thru_hole circle (at 15.24 17.78) (size 2.1 2.1) (drill 1.4) (layers *.Cu *.Mask))
-    (pad 8 thru_hole circle (at 0 17.78) (size 2.1 2.1) (drill 1.4) (layers *.Cu *.Mask))
-    (pad 18 thru_hole circle (at 15.24 15.24) (size 2.1 2.1) (drill 1.4) (layers *.Cu *.Mask))
-    (pad 9 thru_hole circle (at 0 20.32) (size 2.1 2.1) (drill 1.4) (layers *.Cu *.Mask))
-    (pad 19 thru_hole circle (at 15.24 12.7) (size 2.1 2.1) (drill 1.4) (layers *.Cu *.Mask))
+    (pad 7 thru_hole circle (at 0 15.24) (size 2.1 2.1) (drill 1.4) (layers *.Cu *.Mask)
+      (net 23 "Net-(A1-Pad7)"))
+    (pad 17 thru_hole circle (at 15.24 17.78) (size 2.1 2.1) (drill 1.4) (layers *.Cu *.Mask)
+      (net 24 "Net-(A1-Pad17)"))
+    (pad 8 thru_hole circle (at 0 17.78) (size 2.1 2.1) (drill 1.4) (layers *.Cu *.Mask)
+      (net 25 "Net-(A1-Pad8)"))
+    (pad 18 thru_hole circle (at 15.24 15.24) (size 2.1 2.1) (drill 1.4) (layers *.Cu *.Mask)
+      (net 26 "Net-(A1-Pad18)"))
+    (pad 9 thru_hole circle (at 0 20.32) (size 2.1 2.1) (drill 1.4) (layers *.Cu *.Mask)
+      (net 27 "Net-(A1-Pad9)"))
+    (pad 19 thru_hole circle (at 15.24 12.7) (size 2.1 2.1) (drill 1.4) (layers *.Cu *.Mask)
+      (net 28 "Net-(A1-Pad19)"))
     (pad 10 thru_hole circle (at 0 22.86) (size 2.1 2.1) (drill 1.4) (layers *.Cu *.Mask)
       (net 16 INT))
-    (pad 20 thru_hole circle (at 15.24 10.16) (size 2.1 2.1) (drill 1.4) (layers *.Cu *.Mask))
-    (pad 11 thru_hole circle (at 0 25.4) (size 2.1 2.1) (drill 1.4) (layers *.Cu *.Mask))
+    (pad 20 thru_hole circle (at 15.24 10.16) (size 2.1 2.1) (drill 1.4) (layers *.Cu *.Mask)
+      (net 29 "Net-(A1-Pad20)"))
+    (pad 11 thru_hole circle (at 0 25.4) (size 2.1 2.1) (drill 1.4) (layers *.Cu *.Mask)
+      (net 30 "Net-(A1-Pad11)"))
     (pad 21 thru_hole circle (at 15.24 7.62) (size 2.1 2.1) (drill 1.4) (layers *.Cu *.Mask)
       (net 2 +3V3))
@@
     (pad 23 thru_hole circle (at 15.24 2.54) (size 2.1 2.1) (drill 1.4) (layers *.Cu *.Mask)
       (net 1 GND))
-    (pad 24 thru_hole circle (at 15.24 0) (size 2.1 2.1) (drill 1.4) (layers *.Cu *.Mask))
+    (pad 24 thru_hole circle (at 15.24 0) (size 2.1 2.1) (drill 1.4) (layers *.Cu *.Mask)
+      (net 31 "Net-(A1-Pad24)"))
     (model ${KISYS3DMOD}/Module.3dshapes/Sparkfun_Pro_Micro.wrl
       (at (xyz 0 0 0))
@@
   )
   (module Symbol:OSHW-Symbol_6.7x6mm_SilkScreen (layer B.Cu)
-    (at 59.055 100.33 90)
+    (at 59.055 99.695 90)
     (descr "Open Source Hardware Symbol")
     (tags "Logo Symbol OSHW")
@@
     (pad 6 smd rect (at 1.1 0.33 90) (size 1.06 0.4) (layers F.Cu F.Paste F.Mask)
       (net 3 /A))
-    (pad 5 smd rect (at 1.1 0.98 90) (size 1.06 0.4) (layers F.Cu F.Paste F.Mask))
+    (pad 5 smd rect (at 1.1 0.98 90) (size 1.06 0.4) (layers F.Cu F.Paste F.Mask)
+      (net 32 "Net-(U2-Pad5)"))
     (pad 4 smd rect (at -1.1 0.98 90) (size 1.06 0.4) (layers F.Cu F.Paste F.Mask)
       (net 9 "Net-(U2-Pad4)"))
@@
     (pad 12 smd roundrect (at 4.65 2.54) (size 2.05 0.6) (layers F.Cu F.Paste F.Mask) (roundrect_rratio 0.25)
       (net 16 INT))
-    (pad 11 smd roundrect (at 4.65 3.81) (size 2.05 0.6) (layers F.Cu F.Paste F.Mask) (roundrect_rratio 0.25))
-    (pad 10 smd roundrect (at 4.65 5.08) (size 2.05 0.6) (layers F.Cu F.Paste F.Mask) (roundrect_rratio 0.25))
+    (pad 11 smd roundrect (at 4.65 3.81) (size 2.05 0.6) (layers F.Cu F.Paste F.Mask) (roundrect_rratio 0.25)
+      (net 33 "Net-(U3-Pad11)"))
+    (pad 10 smd roundrect (at 4.65 5.08) (size 2.05 0.6) (layers F.Cu F.Paste F.Mask) (roundrect_rratio 0.25)
+      (net 34 "Net-(U3-Pad10)"))
     (pad 9 smd roundrect (at -4.65 5.08) (size 2.05 0.6) (layers F.Cu F.Paste F.Mask) (roundrect_rratio 0.25)
       (net 1 GND))
@@
     (pad 7 smd roundrect (at -4.65 2.54) (size 2.05 0.6) (layers F.Cu F.Paste F.Mask) (roundrect_rratio 0.25)
       (net 8 "Net-(C1-Pad2)"))
-    (pad 6 smd roundrect (at -4.65 1.27) (size 2.05 0.6) (layers F.Cu F.Paste F.Mask) (roundrect_rratio 0.25))
-    (pad 5 smd roundrect (at -4.65 0) (size 2.05 0.6) (layers F.Cu F.Paste F.Mask) (roundrect_rratio 0.25))
-    (pad 4 smd roundrect (at -4.65 -1.27) (size 2.05 0.6) (layers F.Cu F.Paste F.Mask) (roundrect_rratio 0.25))
-    (pad 3 smd roundrect (at -4.65 -2.54) (size 2.05 0.6) (layers F.Cu F.Paste F.Mask) (roundrect_rratio 0.25))
+    (pad 6 smd roundrect (at -4.65 1.27) (size 2.05 0.6) (layers F.Cu F.Paste F.Mask) (roundrect_rratio 0.25)
+      (net 35 "Net-(U3-Pad6)"))
+    (pad 5 smd roundrect (at -4.65 0) (size 2.05 0.6) (layers F.Cu F.Paste F.Mask) (roundrect_rratio 0.25)
+      (net 36 "Net-(U3-Pad5)"))
+    (pad 4 smd roundrect (at -4.65 -1.27) (size 2.05 0.6) (layers F.Cu F.Paste F.Mask) (roundrect_rratio 0.25)
+      (net 37 "Net-(U3-Pad4)"))
+    (pad 3 smd roundrect (at -4.65 -2.54) (size 2.05 0.6) (layers F.Cu F.Paste F.Mask) (roundrect_rratio 0.25)
+      (net 38 "Net-(U3-Pad3)"))
     (pad 2 smd roundrect (at -4.65 -3.81) (size 2.05 0.6) (layers F.Cu F.Paste F.Mask) (roundrect_rratio 0.25)
       (net 9 "Net-(U2-Pad4)"))
@@
   (gr_line (start 67.31 75.565) (end 67.31 104.775) (layer Edge.Cuts) (width 0.1))
   (gr_line (start 49.53 104.775) (end 49.53 75.565) (layer Edge.Cuts) (width 0.1))
-  (gr_text "nerdyscout.github.io/\nProMicro/BUS\nv1.3" (at 58.42 96.52 270) (layer B.SilkS)
+  (gr_text "nerdyscout.github.io/\nProMicro/BUS\nv1.4" (at 58.42 96.52 270) (layer B.SilkS)
     (effects (font (size 1 1) (thickness 0.25)) (justify left mirror))
   )
