File: BUS/ProMicro_BUS.sch (KiCad schematic (older format))
At the start: 17 parts, among them J1 Conn_01x03, U1 MAX3483, U2 MCP2515-xSO, U3 MAX3051, Y1 Crystal

Commit message: dump
Parts:
- removed A1: Sparkfun_Pro_Micro_3V3, Module:Sparkfun_Pro_Micro, symbol MCU_Module:Sparkfun_Pro_Micro_3V3
- removed C1, C5, C6: 100n, Capacitor_SMD:C_0603_1608Metric, symbol Device:C
- removed C4: 10µ, Capacitor_SMD:C_0603_1608Metric, symbol Device:C
- added A1: Sparkfun_Pro_Micro, Module:Sparkfun_Pro_Micro, symbol MCU_Module:Sparkfun_Pro_Micro
- added C2: 100n, Capacitor_SMD:C_0402_1005Metric, symbol Device:C
- added C3: 10µ, Capacitor_SMD:C_0603_1608Metric, symbol Device:C
- C1: renamed from C2; Config (none) -> +canbus,-modbus; Variant canbus -> (none)
- C4: renamed from C3; Config (none) -> +canbus,-modbus; Variant canbus -> (none)
- J1: Config (none) -> modbus, canbus; Variant modbus, canbus -> (none)
- R1, U1: Config (none) -> -canbus,+modbus; Variant modbus -> (none)
- U2: renamed from U3; Config (none) -> +canbus,-modbus; Variant canbus -> (none)
- U3: renamed from U2; Config (none) -> +canbus,-modbus; Variant canbus -> (none)
- Y1: Config (none) -> +canbus,-modbus; Variant canbus -> (none)
- renumbered JP2 to JP1, JP1 to JP2
Connections:
- net labels added: CIPO, COPI, CS0, CS1, INT, RXD, SCK, TXD, ~RST
- net labels removed: A0, A1, A2, A3, D0, D1, D10, D14, D15, D16, D2, D3, D4, D5, D6, D7, D8, D9, Reset
- wire segments 101 -> 84
- no-connect marks 7 -> 18
Other:
- note removed: "CS"
- note removed: "Canbus"
- note removed: "INT"
- note removed: "MISO"
- note removed: "MOSI"
- note removed: "Modbus"
- note removed: "RXD"
- note removed: "SCK"
- note removed: "SCL"
- note removed: "SDA"
- note removed: "TCK"
- note removed: "TDI"
- note removed: "TDO"
- note removed: "TMS"
- note removed: "TXD"
- note removed: "TXDEN"
- note removed: "VBAT"
- moved on the sheet: C1, C4, J1, JP1, JP2, R1, U1, U2, U3, Y1

Commit message: update schematic and PCBs
Parts:
- A1: Config dnp -> (none); Variant (none) -> dnp
- C1, C4, Y1: Config +canbus,-modbus -> (none); Variant (none) -> +canbus,-modbus
- J1: Config modbus, canbus -> (none); Variant (none) -> modbus, canbus
- R1: Config -canbus,+modbus -> (none); Variant (none) -> -canbus,+modbus
- U1: Config -canbus,+modbus -> (none); MPN (none) -> MAX3483ECSA+T; Variant (none) -> -canbus,+modbus; manf# MAX3483ECSA+T -> (none)
- U2: Config +canbus,-modbus -> (none); MPN (none) -> MAX3051EKA+T; Variant (none) -> +canbus,-modbus; manf# MAX3051EKA+T -> (none)
- U3: Config +canbus,-modbus -> (none); MPN (none) -> MCP2515-I/SO; Variant (none) -> +canbus,-modbus; manf# MCP2515-I/SO -> (none)
Changed lines of the file:
@@
 F 2 "Crystal:Crystal_SMD_5032-2Pin_5.0x3.2mm" H 2500 5500 50  0001 C CNN
 F 3 "~" H 2500 5500 50  0001 C CNN
-F 4 "+canbus,-modbus" H 2500 5500 50  0001 C CNN "Config"
+F 4 "+canbus,-modbus" H 2500 5500 50  0001 C CNN "Variant"
 	1    2500 5500
 	0    -1   -1   0
@@
 F 2 "Capacitor_SMD:C_0603_1608Metric" H 2163 5200 50  0001 C CNN
 F 3 "~" H 2125 5350 50  0001 C CNN
-F 4 "+canbus,-modbus" H 2125 5350 50  0001 C CNN "Config"
+F 4 "+canbus,-modbus" H 2125 5350 50  0001 C CNN "Variant"
 	1    2125 5350
 	0    -1   -1   0
@@
 F 2 "Capacitor_SMD:C_0603_1608Metric" H 2163 5500 50  0001 C CNN
 F 3 "~" H 2125 5650 50  0001 C CNN
-F 4 "+canbus,-modbus" H 2125 5650 50  0001 C CNN "Config"
+F 4 "+canbus,-modbus" H 2125 5650 50  0001 C CNN "Variant"
 	1    2125 5650
 	0    1    1    0
@@
 F 2 "Package_SO:SO-8_3.9x4.9mm_P1.27mm" H 3750 1700 50  0001 C CNN
 F 3 "https://datasheets.maximintegrated.com/en/ds/MAX3483-MAX3491.pdf" H 3750 2450 50  0001 C CNN
-F 4 "MAX3483ECSA+T" H 3750 2400 50  0001 C CNN "manf#"
+F 4 "MAX3483ECSA+T" H 3750 2400 50  0001 C CNN "MPN"
 F 5 "C57664" H 3750 2400 50  0001 C CNN "LCSC#"
-F 6 "-canbus,+modbus" H 3750 2400 50  0001 C CNN "Config"
+F 6 "-canbus,+modbus" H 3750 2400 50  0001 C CNN "Variant"
 	1    3750 2400
 	1    0    0    -1
@@
 F 2 "Resistor_SMD:R_0603_1608Metric" V 4430 2450 50  0001 C CNN
 F 3 "~" H 4500 2450 50  0001 C CNN
-F 4 "-canbus,+modbus" H 4500 2450 50  0001 C CNN "Config"
+F 4 "-canbus,+modbus" H 4500 2450 50  0001 C CNN "Variant"
 	1    4500 2450
 	1    0    0    -1
@@
 F 2 "Package_SO:SOIC-18W_7.5x11.6mm_P1.27mm" H 3750 4350 50  0001 C CIN
 F 3 "http://ww1.microchip.com/downloads/en/DeviceDoc/21801e.pdf" H 3850 4450 50  0001 C CNN
-F 4 "MCP2515-I/SO" H 3750 5250 50  0001 C CNN "manf#"
-F 5 "+canbus,-modbus" H 3750 5250 50  0001 C CNN "Config"
+F 4 "MCP2515-I/SO" H 3750 5250 50  0001 C CNN "MPN"
+F 5 "+canbus,-modbus" H 3750 5250 50  0001 C CNN "Variant"
 F 6 "C12368" H 3750 5250 50  0001 C CNN "LCSC#"
 	1    3750 5250
@@
 F 2 "Package_TO_SOT_SMD:SOT-23-8" H 6250 4850 50  0001 C CIN
 F 3 "http://datasheets.maximintegrated.com/en/ds/MAX3051.pdf" H 6250 4850 50  0001 C CNN
-F 4 "+canbus,-modbus" H 6250 4850 50  0001 C CNN "Config"
-F 5 "MAX3051EKA+T" H 6250 4850 50  0001 C CNN "manf#"
+F 4 "+canbus,-modbus" H 6250 4850 50  0001 C CNN "Variant"
+F 5 "MAX3051EKA+T" H 6250 4850 50  0001 C CNN "MPN"
 F 6 "C112005" H 6250 4850 50  0001 C CNN "LCSC#"
 	1    6250 4850
@@
 F 2 "TerminalBlock_TE-Connectivity:TerminalBlock_TE_282834-3_1x03_P2.54mm_Horizontal" H 5200 2400 50  0001 C CNN
 F 3 "~" H 5200 2400 50  0001 C CNN
-F 4 "modbus, canbus" H 5200 2400 50  0001 C CNN "Config"
+F 4 "modbus, canbus" H 5200 2400 50  0001 C CNN "Variant"
 	1    5200 2400
 	1    0    0    -1
@@
 F 2 "Module:Sparkfun_Pro_Micro" H 9850 1650 50  0001 L CNN
 F 3 "https://cdn.sparkfun.com/datasheets/Dev/Arduino/Boards/Pro_Micro_v13b.pdf" H 9750 2200 50  0001 C CNN
-F 4 "dnp" H 9750 3000 50  0001 C CNN "Config"
+F 4 "dnp" H 9750 3000 50  0001 C CNN "Variant"
 	1    9750 3000
 	1    0    0    -1

Commit message: update PCBs to be stackable
Parts:
- A1: symbol MCU_Module:Sparkfun_Pro_Micro -> ProMicro:Sparkfun_Pro_Micro
Changed lines of the file:
@@
 $EndComp
 $Comp
-L MCU_Module:Sparkfun_Pro_Micro A1
+L ProMicro:Sparkfun_Pro_Micro A1
 U 1 1 5F84D072
 P 9750 3000

Commit message: BUS
Changed lines of the file:
@@
 	1500 2250 1500 1500
-Wire Wire Line
-	9950 1700 9950 1800
 Wire Wire Line
 	10000 5200 10000 5350
@@
 	1    0    0    -1
 $EndComp
-Wire Wire Line
-	9750 4400 9750 4300
 Text GLabel 9125 3500 0    50   Input ~ 0
 TXD
@@
 NoConn ~ 9250 3900
 NoConn ~ 9250 3800
+Wire Wire Line
+	9950 1700 9950 1800
+Wire Wire Line
+	9750 4300 9750 4400
 $EndSCHEMATC

Commit message: blindly dumped everything
Parts:
- added JP4: SolderJumper_2_Open, Jumper:SolderJumper-2_P1.3mm_Open_RoundedPad1.0x1.5mm, symbol Jumper:SolderJumper_2_Open
Connections:
- net INT: now also JP4.2 (B); no longer U3.12 (~INT)
- new net: JP4.1 (A), U3.12 (~INT)
Changed lines of the file:
@@
 encoding utf-8
 Sheet 1 1
-Title "ProMicro_BUS"
+Title "BUS"
 Date "2020-10-12"
 Rev "v1.3"
-Comp ""
+Comp "nerdsycout"
 Comment1 ""
 Comment2 ""
@@
 	7750 5500 8100 5500
 Wire Wire Line
-	4350 5250 4625 5250
+	4900 5250 5175 5250
 Wire Wire Line
 	4350 5850 4625 5850
@@
 Text GLabel 4625 5850 2    50   Input ~ 0
 ~RST
-Text GLabel 4625 5250 2    50   Input ~ 0
+Text GLabel 5175 5250 2    50   Input ~ 0
 INT
 Text GLabel 2875 4650 0    50   Input ~ 0
@@
 Wire Wire Line
 	9750 4300 9750 4400
+$Comp
+L Jumper:SolderJumper_2_Open JP4
+U 1 1 608F494F
+P 4750 5250
+F 0 "JP4" H 4750 5363 50  0000 C CNN
+F 1 "SolderJumper_2_Open" H 4750 5364 50  0001 C CNN
+F 2 "Jumper:SolderJumper-2_P1.3mm_Open_RoundedPad1.0x1.5mm" H 4750 5250 50  0001 C CNN
+F 3 "~" H 4750 5250 50  0001 C CNN
+	1    4750 5250
+	1    0    0    -1
+$EndComp
+Wire Wire Line
+	4600 5250 4350 5250
 $EndSCHEMATC
