File: QWIIC/ProMicro_QWIIC.sch (KiCad schematic (older format))
At the start: 19 parts, among them J1 Qwiic, J2 Qwiic, J3 Conn_01x02, J4 Conn_01x02, J5 Conn_01x03, J6 Conn_01x03, U1 ADS1015IDGS, U2 BME280

Commit message: update schematic and PCBs
Parts:
- R3, R4: MPN (none) -> RC0402FR-074K7L; manf# RC0402FR-074K7L -> (none)
Changed lines of the file:
@@
 F 2 "Resistor_SMD:R_0603_1608Metric" V 8930 5500 50  0001 C CNN
 F 3 "~" H 9000 5500 50  0001 C CNN
-F 4 "RC0402FR-074K7L" H 9000 5500 50  0001 C CNN "manf#"
+F 4 "RC0402FR-074K7L" H 9000 5500 50  0001 C CNN "MPN"
 	1    9000 5500
 	-1   0    0    1
@@
 F 2 "Resistor_SMD:R_0603_1608Metric" V 9430 5500 50  0001 C CNN
 F 3 "~" H 9500 5500 50  0001 C CNN
-F 4 "RC0402FR-074K7L" H 9500 5500 50  0001 C CNN "manf#"
+F 4 "RC0402FR-074K7L" H 9500 5500 50  0001 C CNN "MPN"
 F 5 "C105871" H 9500 5500 50  0001 C CNN "lcsc#"
 	1    9500 5500

Commit message: update PCBs to be stackable
Parts:
- A1: symbol MCU_Module:Sparkfun_Pro_Micro_3V3 -> ProMicro:Sparkfun_Pro_Micro
Changed lines of the file:
@@
 BTN
 $Comp
-L MCU_Module:Sparkfun_Pro_Micro_3V3 A1
+L ProMicro:Sparkfun_Pro_Micro A1
 U 1 1 5ED4BC58
-P 8900 3000
-F 0 "A1" H 8550 3975 50  0000 C CNN
-F 1 "Sparkfun_Pro_Micro_3V3" H 9500 2025 50  0000 C CNN
-F 2 "Module:Sparkfun_Pro_Micro" H 8900 3000 50  0001 C CIN
-F 3 "https://www.sparkfun.com/products/12587" H 8900 2000 50  0001 C CNN
-	1    8900 3000
+P 10650 3000
+F 0 "A1" H 10300 3975 50  0000 C CNN
+F 1 "Sparkfun_Pro_Micro_3V3" H 11250 2025 50  0000 C CNN
+F 2 "Module:Sparkfun_Pro_Micro" H 10650 3000 50  0001 C CIN
+F 3 "https://www.sparkfun.com/products/12587" H 10650 2000 50  0001 C CNN
+	1    10650 3000
 	1    0    0    -1
 $EndComp
