File: LOG/ProMicro_LOG.sch (KiCad schematic (older format))
At the start: 16 parts, among them J1 Micro_SD_Card_Det, U1 DS3231MZ

Commit message: dump
Parts:
- removed A1: Sparkfun_Pro_Micro_3V3, Module:Sparkfun_Pro_Micro, symbol MCU_Module:Sparkfun_Pro_Micro_3V3
- added A1: Sparkfun_Pro_Micro, Module:Sparkfun_Pro_Micro, symbol MCU_Module:Sparkfun_Pro_Micro
- D1, J1: Config (none) -> -RTC,+LOG
- JP1: renamed from JP2; symbol Device:Jumper_NO_Small -> ProMicro_LOG-rescue:Jumper_NO_Small-Device
- JP2: renamed from JP1; symbol Device:Jumper_NO_Small -> ProMicro_LOG-rescue:Jumper_NO_Small-Device
- R1: renamed from R6; Config (none) -> -RTC,+LOG
- R2: renamed from R1; Config (none) -> +RTC,-LOG
- R3: renamed from R2; Config (none) -> +RTC,-LOG
- R4: renamed from R5; Config (none) -> -RTC,+LOG
- R5: renamed from R3; Config (none) -> +RTC,-LOG
- R6: renamed from R4; Config (none) -> +RTC,-LOG
- U1: Config (none) -> +RTC,-LOG
- renumbered JP4 to JP3
Connections:
- net labels added: PWM, ~RST
- net labels removed: Reset, TRG
- wire segments 59 -> 56
- no-connect marks 12 -> 11
Other:
- note added: "TCK"
- note added: "TD0"
- note added: "TDI"
- note added: "TMS"
- moved on the sheet: D1, J1, JP1, JP2, JP3, R1, R2, R3, R4, U1

Commit message: clean
Parts:
- A1: symbol MCU_Module:Sparkfun_Pro_Micro -> ProMicro_LOG-rescue:Sparkfun_Pro_Micro-MCU_Module
Changed lines of the file:
@@
 SDA
 $Comp
-L MCU_Module:Sparkfun_Pro_Micro A1
+L ProMicro_LOG-rescue:Sparkfun_Pro_Micro-MCU_Module A1
 U 1 1 5F84D072
 P 9750 3000

Commit message: update schematic and PCBs
Parts:
- A1: Config dnp -> (none); Variant (none) -> dnp
- D1, J1, R1, R4: Config -RTC,+LOG -> (none); Variant (none) -> -RTC,+LOG
- R2, R3, R5, R6, U1: Config +RTC,-LOG -> (none); Variant (none) -> +RTC,-LOG
Changed lines of the file:
@@
 F 2 "Connector_Card:microSD_HC_Molex_104031-0811" H 5500 3400 50  0001 C CNN
 F 3 "https://www.hirose.com/product/en/download_file/key_name/DM3/category/Catalog/doc_file_id/49662/?file_category_id=4&item_id=195&is_series=1" H 3450 2800 50  0001 C CNN
-F 4 "-RTC,+LOG" H 3450 2700 50  0001 C CNN "Config"
+F 4 "-RTC,+LOG" H 3450 2700 50  0001 C CNN "Variant"
 	1    3450 2700
 	1    0    0    -1
@@
 F 2 "Package_SO:SOIC-8_3.9x4.9mm_P1.27mm" H 3250 4700 50  0001 C CNN
 F 3 "http://datasheets.maximintegrated.com/en/ds/DS3231M.pdf" H 3250 4600 50  0001 C CNN
-F 4 "+RTC,-LOG" H 3250 5200 50  0001 C CNN "Config"
+F 4 "+RTC,-LOG" H 3250 5200 50  0001 C CNN "Variant"
 	1    3250 5200
 	1    0    0    -1
@@
 F 2 "Resistor_SMD:R_0603_1608Metric" V 8930 5500 50  0001 C CNN
 F 3 "~" H 9000 5500 50  0001 C CNN
-F 4 "+RTC,-LOG" H 9000 5500 50  0001 C CNN "Config"
+F 4 "+RTC,-LOG" H 9000 5500 50  0001 C CNN "Variant"
 	1    9000 5500
 	1    0    0    -1
@@
 F 2 "Resistor_SMD:R_0603_1608Metric" V 9430 5500 50  0001 C CNN
 F 3 "~" H 9500 5500 50  0001 C CNN
-F 4 "+RTC,-LOG" H 9500 5500 50  0001 C CNN "Config"
+F 4 "+RTC,-LOG" H 9500 5500 50  0001 C CNN "Variant"
 	1    9500 5500
 	1    0    0    -1
@@
 F 2 "Resistor_SMD:R_0603_1608Metric" V 3930 4700 50  0001 C CNN
 F 3 "~" H 4000 4700 50  0001 C CNN
-F 4 "+RTC,-LOG" H 4000 4700 50  0001 C CNN "Config"
+F 4 "+RTC,-LOG" H 4000 4700 50  0001 C CNN "Variant"
 	1    4000 4700
 	1    0    0    -1
@@
 F 2 "Resistor_SMD:R_0603_1608Metric" V 4305 4700 50  0001 C CNN
 F 3 "~" H 4375 4700 50  0001 C CNN
-F 4 "+RTC,-LOG" H 4375 4700 50  0001 C CNN "Config"
+F 4 "+RTC,-LOG" H 4375 4700 50  0001 C CNN "Variant"
 	1    4375 4700
 	1    0    0    -1
@@
 F 2 "Resistor_SMD:R_0603_1608Metric" V 8430 5300 50  0001 C CNN
 F 3 "~" H 8500 5300 50  0001 C CNN
-F 4 "-RTC,+LOG" H 8500 5300 50  0001 C CNN "Config"
+F 4 "-RTC,+LOG" H 8500 5300 50  0001 C CNN "Variant"
 	1    8500 5300
 	1    0    0    -1
@@
 F 2 "LED_SMD:LED_0603_1608Metric" H 8500 5675 50  0001 C CNN
 F 3 "~" H 8500 5675 50  0001 C CNN
-F 4 "-RTC,+LOG" H 8500 5675 50  0001 C CNN "Config"
+F 4 "-RTC,+LOG" H 8500 5675 50  0001 C CNN "Variant"
 	1    8500 5675
 	0    -1   -1   0
@@
 F 2 "Resistor_SMD:R_0603_1608Metric" V 2055 3200 50  0001 C CNN
 F 3 "~" H 2125 3200 50  0001 C CNN
-F 4 "-RTC,+LOG" H 2125 3200 50  0001 C CNN "Config"
+F 4 "-RTC,+LOG" H 2125 3200 50  0001 C CNN "Variant"
 	1    2125 3200
 	0    1    1    0
@@
 F 2 "Module:Sparkfun_Pro_Micro" H 9850 1650 50  0001 L CNN
 F 3 "https://cdn.sparkfun.com/datasheets/Dev/Arduino/Boards/Pro_Micro_v13b.pdf" H 9750 2200 50  0001 C CNN
-F 4 "dnp" H 9750 3000 50  0001 C CNN "Config"
+F 4 "dnp" H 9750 3000 50  0001 C CNN "Variant"
 	1    9750 3000
 	1    0    0    -1

Commit message: merged libs into one
Parts:
- A1: symbol ProMicro_LOG-rescue:Sparkfun_Pro_Micro-MCU_Module -> ProMicro:Sparkfun_Pro_Micro; Variant dnp -> DNP
- JP1, JP2: symbol ProMicro_LOG-rescue:Jumper_NO_Small-Device -> Device:Jumper_NO_Small
Changed lines of the file:
@@
 	3250 5700 3250 5600
 $Comp
-L ProMicro_LOG-rescue:Jumper_NO_Small-Device JP2
+L Device:Jumper_NO_Small JP2
 U 1 1 5EB76258
 P 4625 5300
@@
 	4000 4850 4000 5300
 $Comp
-L ProMicro_LOG-rescue:Jumper_NO_Small-Device JP1
+L Device:Jumper_NO_Small JP1
 U 1 1 5EB83C6F
 P 4625 5000
@@
 SDA
 $Comp
-L ProMicro_LOG-rescue:Sparkfun_Pro_Micro-MCU_Module A1
+L ProMicro:Sparkfun_Pro_Micro A1
 U 1 1 5F84D072
 P 9750 3000
@@
 F 2 "Module:Sparkfun_Pro_Micro" H 9850 1650 50  0001 L CNN
 F 3 "https://cdn.sparkfun.com/datasheets/Dev/Arduino/Boards/Pro_Micro_v13b.pdf" H 9750 2200 50  0001 C CNN
-F 4 "dnp" H 9750 3000 50  0001 C CNN "Variant"
+F 4 "DNP" H 9750 3000 50  0001 C CNN "Variant"
 	1    9750 3000
 	1    0    0    -1
