File: LORA/ProMicro_LORA.sch (KiCad schematic (older format))
At the start: 44 parts, among them J1 SMA, J2 COAX, U1 SX1276, U2 AS179-92LF, Y1 32Mhz

Commit message: dump
Parts:
- removed A1: Sparkfun_Pro_Micro_3V3, Module:Sparkfun_Pro_Micro, symbol MCU_Module:Sparkfun_Pro_Micro_3V3
- added A1: Sparkfun_Pro_Micro, Module:Sparkfun_Pro_Micro, symbol MCU_Module:Sparkfun_Pro_Micro
- C10, C11: Config (none) -> DNP
- U1: symbol RF:SX1276 -> ProMicro_LORA-rescue:SX1276-RF
Connections:
- net labels added: CIPO, COPI, CS0, DIO0, DIO1, RFRST, SCK
- net labels removed: D10, D14, D15, D16, D5, D7, D8
- wire segments 137 -> 134
- no-connect marks 18 -> 17
Other:
- note removed: "BTN"
- note removed: "CS0"
- note removed: "CS1"
- note removed: "DIO0"
- note removed: "DIO1"
- note removed: "INT0"
- note removed: "Reset"
- note removed: "SCK"
- note removed: "SDI"
- note removed: "SDO"
- note removed: "TODO: hier muss wohl eine Spannung ran"
- note removed: "VBAT/2"
- moved on the sheet: C22, C23, TP5, TP6

Commit message: clean
Parts:
- A1: symbol MCU_Module:Sparkfun_Pro_Micro -> ProMicro_LORA-rescue:Sparkfun_Pro_Micro-MCU_Module
Changed lines of the file:
@@
 $EndComp
 $Comp
-L MCU_Module:Sparkfun_Pro_Micro A1
+L ProMicro_LORA-rescue:Sparkfun_Pro_Micro-MCU_Module A1
 U 1 1 5F84D072
 P 9750 3000

Commit message: update schematic and PCBs
Parts:
- A1, C10, C11: Config DNP -> (none); Variant (none) -> DNP
- C1, C4: MPN (none) -> 0402CG150J500NT; manf# 0402CG150J500NT -> (none)
- C12: MPN (none) -> CL05C1R2BB5NNNC; manf# CL05C1R2BB5NNNC -> (none)
- C13, C14: MPN (none) -> 0402B102K500NT; manf# 0402B102K500NT -> (none)
- C15, C18, C7, C9: MPN (none) -> 0402CG470J500NT; manf# 0402CG470J500NT -> (none)
- C16, C17, C19, C20, C21: MPN (none) -> CL05B104KO5NNNC; manf# CL05B104KO5NNNC -> (none)
- C2: MPN (none) -> 0402CG1R5C500NT; manf# 0402CG1R5C500NT -> (none)
- C22: MPN (none) -> CL05A105KA5NQNC; manf# CL05A105KA5NQNC -> (none)
- C23: MPN (none) -> CL05A106MQ5NUNC; manf# CL05A106MQ5NUNC -> (none)
- C3: MPN (none) -> 0402CG330J500NT; manf# 0402CG330J500NT -> (none)
- C5: MPN (none) -> 0402CG4R7C500NT; manf# 0402CG4R7C500NT -> (none)
- C6: MPN (none) -> 0402CG3R3C500NT; manf# 0402CG3R3C500NT -> (none)
- L1: symbol pspice:INDUCTOR -> Device:L; MPN (none) -> HK100533NJ-T; manf# HK100533NJ-T -> (none)
- L2, L3: symbol pspice:INDUCTOR -> Device:L; MPN (none) -> SDCL1005C10NJTDF; manf# SDCL1005C10NJTDF -> (none)
- L4: symbol pspice:INDUCTOR -> Device:L; MPN (none) -> MLG1005S6N2ST000; manf# MLG1005S6N2ST000 -> (none)
- L5: symbol pspice:INDUCTOR -> Device:L; MPN (none) -> 0402WGF0000TCE; manf# 0402WGF0000TCE -> (none)
- R1: MPN (none) -> 0402WGF1001TCE; manf# 0402WGF1001TCE -> (none)
- U1: symbol ProMicro_LORA-rescue:SX1276-RF -> RF:SX1276
- U2: MPN (none) -> AS179-92LF; manf# AS179-92LF -> (none)
- Y1: MPN (none) -> X1E000021016300; manf# X1E000021016300 -> (none)
Other:
- moved on the sheet: JP1, TP2, TP3, TP4

Commit message: fixed lib
Parts:
- A1: symbol ProMicro_LORA-rescue:Sparkfun_Pro_Micro-MCU_Module -> ProMicro:Sparkfun_Pro_Micro
- U1: symbol RF:SX1276 -> sx1276:SX1276
Other:
- moved on the sheet: JP1, TP2, TP3, TP4
Changed lines of the file:
@@
 	3500 5150 3500 5350
 Wire Wire Line
-	3400 3150 3200 3150
-Wire Wire Line
 	1475 5150 1250 5150
 Wire Wire Line
@@
 	3000 2850 3400 2850
 Wire Wire Line
-	5000 3450 4600 3450
-Wire Wire Line
-	5000 3550 4600 3550
+	3000 3250 3400 3250
+Wire Wire Line
+	3000 3350 3400 3350
 Wire Wire Line
 	3000 3850 3400 3850
@@
 	3500 4750 3500 5150
 Wire Wire Line
-	3400 3250 3000 3250
-Wire Wire Line
-	3400 3350 3000 3350
-Wire Wire Line
-	3400 3550 3000 3550
+	4600 3350 5000 3350
+Wire Wire Line
+	4600 3450 5000 3450
+Wire Wire Line
+	4600 3650 5000 3650
 Wire Wire Line
 	3250 2000 3800 2000
@@
 Text GLabel 1000 6250 0    50   Input ~ 0
 RFI-HF
-Text GLabel 5000 3450 2    50   Input ~ 0
+Text GLabel 3000 3250 0    50   Input ~ 0
 RFO_HF
-Text GLabel 5000 3550 2    50   Input ~ 0
+Text GLabel 3000 3350 0    50   Input ~ 0
 RFI-HF
 Text GLabel 6000 2950 2    50   Input ~ 0
@@
 L Connector:TestPoint TP2
 U 1 1 5E1AA0A9
-P 3000 3250
-F 0 "TP2" V 3000 3450 50  0000 L CNN
-F 1 "DIO2" V 3000 3450 50  0001 L CNN
-F 2 "TestPoint:TestPoint_Pad_D1.0mm" H 3200 3250 50  0001 C CNN
-F 3 "~" H 3200 3250 50  0001 C CNN
-	1    3000 3250
-	0    -1   -1   0
+P 5000 3350
+F 0 "TP2" V 5000 3550 50  0000 L CNN
+F 1 "DIO2" V 5000 3550 50  0001 L CNN
+F 2 "TestPoint:TestPoint_Pad_D1.0mm" H 5200 3350 50  0001 C CNN
+F 3 "~" H 5200 3350 50  0001 C CNN
+	1    5000 3350
+	0    1    -1   0
 $EndComp
 $Comp
 L Connector:TestPoint TP3
 U 1 1 5E1AA436
-P 3000 3350
-F 0 "TP3" V 3000 3550 50  0000 L CNN
-F 1 "DIO3" V 3000 3550 50  0001 L CNN
-F 2 "TestPoint:TestPoint_Pad_D1.0mm" H 3200 3350 50  0001 C CNN
-F 3 "~" H 3200 3350 50  0001 C CNN
-	1    3000 3350
-	0    -1   -1   0
+P 5000 3450
+F 0 "TP3" V 5000 3650 50  0000 L CNN
+F 1 "DIO3" V 5000 3650 50  0001 L CNN
+F 2 "TestPoint:TestPoint_Pad_D1.0mm" H 5200 3450 50  0001 C CNN
+F 3 "~" H 5200 3450 50  0001 C CNN
+	1    5000 3450
+	0    1    -1   0
 $EndComp
 $Comp
 L Connector:TestPoint TP4
 U 1 1 5E1AA6B5
-P 3000 3550
-F 0 "TP4" V 3000 3750 50  0000 L CNN
-F 1 "DIO5" V 3000 3750 50  0001 L CNN
-F 2 "TestPoint:TestPoint_Pad_D1.0mm" H 3200 3550 50  0001 C CNN
-F 3 "~" H 3200 3550 50  0001 C CNN
-	1    3000 3550
-	0    -1   -1   0
+P 5000 3650
+F 0 "TP4" V 5000 3850 50  0000 L CNN
+F 1 "DIO5" V 5000 3850 50  0001 L CNN
+F 2 "TestPoint:TestPoint_Pad_D1.0mm" H 5200 3650 50  0001 C CNN
+F 3 "~" H 5200 3650 50  0001 C CNN
+	1    5000 3650
+	0    1    -1   0
 $EndComp
 $Comp
@@
 L Jumper:SolderJumper_2_Open JP1
 U 1 1 5E32FE28
-P 3050 3150
-F 0 "JP1" H 3200 3225 50  0000 C CNN
-F 1 "SolderJumper_2_Open" H 3085 3310 50  0001 C CNN
-F 2 "Jumper:SolderJumper-2_P1.3mm_Open_RoundedPad1.0x1.5mm" H 3050 3150 50  0001 C CNN
-F 3 "~" H 3050 3150 50  0001 C CNN
-	1    3050 3150
-	-1   0    0    1
+P 4900 3250
+F 0 "JP1" H 5050 3325 50  0000 C CNN
+F 1 "SolderJumper_2_Open" H 4935 3410 50  0001 C CNN
+F 2 "Jumper:SolderJumper-2_P1.3mm_Open_RoundedPad1.0x1.5mm" H 4900 3250 50  0001 C CNN
+F 3 "~" H 4900 3250 50  0001 C CNN
+	1    4900 3250
+	1    0    0    -1
 $EndComp
 $Comp
@@
 	6500 5250 6500 5600
 $Comp
-L RF:SX1276 U1
+L sx1276:SX1276 U1
 U 1 1 5EDDF92E
 P 4000 3250
@@
 $EndComp
 $Comp
-L ProMicro_LORA-rescue:Sparkfun_Pro_Micro-MCU_Module A1
+L ProMicro:Sparkfun_Pro_Micro A1
 U 1 1 5F84D072
 P 9750 3000
@@
 Text GLabel 3000 3750 0    50   Input ~ 0
 SCK
-Text GLabel 2750 3050 0    50   Input ~ 0
+Text GLabel 4700 3150 2    50   Input ~ 0
 DIO0
-Text GLabel 2675 3150 0    50   Input ~ 0
+Text GLabel 5275 3250 2    50   Input ~ 0
 DIO1
 Wire Wire Line
-	2675 3150 2900 3150
-Wire Wire Line
-	3400 3050 2750 3050
+	5275 3250 5050 3250
 Text GLabel 3000 2850 0    50   Input ~ 0
 RFRST
@@
 Wire Wire Line
 	2400 6250 2750 6250
-NoConn ~ 3400 3450
-NoConn ~ 4600 3350
-NoConn ~ 4600 3250
-Wire Wire Line
-	4600 3850 5500 3850
-Wire Wire Line
-	5500 3850 5500 4850
+Wire Wire Line
+	4600 3950 5500 3950
+Wire Wire Line
+	5500 3950 5500 4850
+Wire Wire Line
+	4700 3150 4600 3150
+Wire Wire Line
+	4600 3250 4750 3250
+NoConn ~ 4600 3550
+NoConn ~ 3400 3150
+NoConn ~ 3400 3050
 $EndSCHEMATC

Commit message: merged libs into one
Parts:
- U1: symbol sx1276:SX1276 -> ProMicro:SX1276
Changed lines of the file:
@@
 	6500 5250 6500 5600
 $Comp
-L sx1276:SX1276 U1
+L ProMicro:SX1276 U1
 U 1 1 5EDDF92E
 P 4000 3250
