File: LORA/LORA.kicad_pcb (KiCad board)
At the start: 4 copper layers, 30.5 x 17.8 mm, 44 parts, among them J1 SMA, J2 COAX, U1 SX1276, U2 AS179-92LF, Y1 32Mhz

Commit message: major cleanup and fixes
Parts:
- moved C14 92.6 mm to (226.3, 86.5)
- moved A1 91.5 mm to (205.3, 81.4)
- moved C1 91.5 mm to (209.1, 84.0)
- moved C17 91.5 mm to (210.9, 92.2)
- moved C18 91.5 mm to (217.4, 84.6)
- moved C19 91.5 mm to (217.4, 85.9)
- moved C20 91.5 mm to (215.5, 85.2)
- moved C22 91.5 mm to (210.9, 93.5)
- moved C4 91.5 mm to (215.6, 83.5)
- moved TP5 91.5 mm to (205.3, 86.2)
- moved TP6 91.5 mm to (205.3, 91.9)
- moved U1 91.5 mm to (215.5, 90.3)
- moved C10 91.5 mm to (228.8, 91.8)
- moved C11 91.5 mm to (228.8, 87.2)
- moved C12 91.5 mm to (222.4, 87.2)
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Connections:
- A1 pad 1: (no net) -> unconnected-(A1-TX/D1-Pad1)
- A1 pad 12: (no net) -> unconnected-(A1-D9/A9-Pad12)
- A1 pad 17: (no net) -> unconnected-(A1-TDI/A0-Pad17)
- A1 pad 18: (no net) -> unconnected-(A1-TDO/A1-Pad18)
- A1 pad 19: (no net) -> unconnected-(A1-TMS/A2-Pad19)
- A1 pad 2: (no net) -> unconnected-(A1-RX/D0-Pad2)
- A1 pad 20: (no net) -> unconnected-(A1-TCK/A3-Pad20)
- A1 pad 22: (no net) -> unconnected-(A1-~{RESET}-Pad22)
- A1 pad 24: (no net) -> unconnected-(A1-RAW-Pad24)
- A1 pad 5: (no net) -> unconnected-(A1-SDA/D2-Pad5)
- A1 pad 6: (no net) -> unconnected-(A1-SCL/D3-Pad6)
- A1 pad 7: (no net) -> unconnected-(A1-D4/A6-Pad7)
- A1 pad 9: (no net) -> unconnected-(A1-D6/A7-Pad9)
- U1 pad 1: (no net) -> unconnected-(U1-RFI_LF-Pad1)
- U1 pad 12: (no net) -> unconnected-(U1-DIO4-Pad12)
- U1 pad 27: (no net) -> unconnected-(U1-PA_BOOST-Pad27)
- U1 pad 28: (no net) -> unconnected-(U1-RFO_LF-Pad28)
Routing:
- net +3V3: track 30.9 -> 8.09 mm, vias 6 -> 4
- net RFRST: track 22.4 -> 21.1 mm
- added copper zone on In2.Cu, net +3V3
- removed copper zone on In2.Cu, net GND
Other:
- net class Default removed
- net class Power removed
- net class small removed
- net class tiny removed
- board text added: "0"
- board text added: "0 mm"
- board text added: "0,01 mm"
- board text added: "0,0152 mm"
- board text added: "0,02"
- board text added: "0,035 mm"
- board text added: "0,1250 mm / 0,0000 mm"
- board text added: "0,2000 mm"
- board text added: "0,2104 mm"
- board text added: "0,25 mm"
- board text added: "0,7912 mm"
- board text added: "1"
- board text added: "3,3"
- board text added: "30,4800 mm x 17,7800 mm"
- board text added: "4"
- board text added: "4,5"
- board text added: "B.Cu"
- board text added: "B.Mask"
- board text added: "B.Paste"
- board text added: "B.Silkscreen"
- board text added: "BOARD CHARACTERISTICS"
- board text added: "Board Thickness:"
- board text added: "Board overall dimensions:"
- board text added: "Bottom Silk Screen"
- board text added: "Bottom Solder Mask"
- board text added: "Bottom Solder Paste"
- board text added: "Castellated pads:"
- board text added: "Color"
- board text added: "Copper Finish:"
- board text added: "Copper Layer Count:"
- board text added: "Dielectric"
- board text added: "Edge card connectors:"
- board text added: "Epsilon R"
- board text added: "F.Cu"
- board text added: "F.Mask"
- board text added: "F.Paste"
- board text added: "F.Silkscreen"
- board text added: "FR4"
- board text added: "Impedance Control:"
- board text added: "In1.Cu"
- board text added: "In2.Cu"
- board text added: "Layer Name"
- board text added: "Loss Tangent"
- board text added: "Material"
- board text added: "Min hole diameter:"
- board text added: "Min track/spacing:"
- board text added: "No"
- board text added: "None"
- board text added: "Not specified"
- board text added: "Plated Board Edge:"
- board text added: "Thickness (mm)"
- board text added: "Top Silk Screen"
- board text added: "Top Solder Mask"
- board text added: "Top Solder Paste"
- board text added: "Type"
- board text added: "Yes"
- board text added: "copper"
- board text added: "core"
- board text added: "prepreg"
