File: BOOST/ProMicro_BOOST.sch (KiCad schematic (older format))
At the start: 24 parts, among them J1 JST, U1 MCP73831-2-OT, U2 TPS61090

Commit message: dump
Parts:
- removed A1: Sparkfun_Pro_Micro_3V3, Module:Sparkfun_Pro_Micro, symbol MCU_Module:Sparkfun_Pro_Micro_3V3
- added A1: Sparkfun_Pro_Micro, Module:Sparkfun_Pro_Micro, symbol MCU_Module:Sparkfun_Pro_Micro
- added LOGO1: Logo_Open_Hardware_Small, Symbol:OSHW-Symbol_6.7x6mm_SilkScreen, symbol Graphic:Logo_Open_Hardware_Small
- C1, C2, D1, J1, U1, U2: Config (none) -> 3V3, 5V; Variant 3V3, 5V -> (none)
Connections:
- net +3V3: now also A1.21 (VCC)
- net GND: now also A1.23 (GND), A1.3 (GND), A1.4 (GND)
- net STAT: now also A1.7 (D4/A6)
- new net +5V: A1.24 (RAW)
- no-connect marks 2 -> 19
Other:
- moved on the sheet: C1, C2, C3, C4, C5, C6, C7, D1, F1, J1, JP1, L1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

Commit message: clean
Parts:
- A1: symbol MCU_Module:Sparkfun_Pro_Micro -> ProMicro_BOOST-rescue:Sparkfun_Pro_Micro-MCU_Module
Connections:
- net labels removed: +5V
Changed lines of the file:
@@
 $EndComp
 $Comp
-L MCU_Module:Sparkfun_Pro_Micro A1
+L ProMicro_BOOST-rescue:Sparkfun_Pro_Micro-MCU_Module A1
 U 1 1 5F84D072
 P 3500 5875
@@
 Wire Wire Line
 	3800 4575 3800 4675
-$Comp
-L power:+5V #PWR01
-U 1 1 5F84FBAC
-P 3800 4575
-F 0 "#PWR01" H 3800 4425 50  0001 C CNN
-F 1 "+5V" V 3800 4825 50  0000 C CNN
-F 2 "" H 3800 4575 50  0001 C CNN
-F 3 "" H 3800 4575 50  0001 C CNN
-	1    3800 4575
-	1    0    0    -1
-$EndComp
 Wire Wire Line
 	3500 7275 3500 7175
@@
 NoConn ~ 3000 5375
 NoConn ~ 3000 5275
+$Comp
+L power:VBUS #PWR?
+U 1 1 5F9D96E1
+P 3800 4575
+F 0 "#PWR?" H 3800 4425 50  0001 C CNN
+F 1 "VBUS" V 3800 4850 50  0000 C CNN
+F 2 "" H 3800 4575 50  0001 C CNN
+F 3 "" H 3800 4575 50  0001 C CNN
+	1    3800 4575
+	1    0    0    -1
+$EndComp
 $EndSCHEMATC

Commit message: update schematic and PCBs
Parts:
- C1: Config 3V3, 5V -> (none); MPN (none) -> CL10A106KP8NNNC; Variant (none) -> 3V3, 5V; manf# CL10A106KP8NNNC -> (none)
- C2: Config 3V3, 5V -> (none); MPN (none) -> C0603C104M4RACTU; Variant (none) -> 3V3, 5V; manf# C0603C104M4RACTU -> (none)
- C3, C7: MPN (none) -> CL10A475KO8NNNC; manf# CL10A475KO8NNNC -> (none)
- C4: MPN (none) -> CL10A106KP8NNNC; manf# CL10A106KP8NNNC -> (none)
- C5: MPN (none) -> C0603C104M4RACTU; manf# C0603C104M4RACTU -> (none)
- C6: MPN (none) -> C0603X105K9RACAUTO; manf# C0603X105K9RACAUTO -> (none)
- D1, J1: Config 3V3, 5V -> (none); Variant (none) -> 3V3, 5V
- F1: MPN (none) -> 04000025WR; manf# 04000025WR -> (none)
- L1: MPN (none) -> 744787068; manf# 744787068 -> (none)
- R1, R2, R6: MPN (none) -> 0603WAF3903T5E; manf# 0603WAF3903T5E -> (none)
- R3: MPN (none) -> 0603WAF2001T5E; manf# 0603WAF2001T5E -> (none)
- R4, R8: MPN (none) -> 0603WAF2003T5E; manf# 0603WAF2003T5E -> (none)
- R5: MPN (none) -> WR06W2404FTL; manf# WR06W2404FTL -> (none)
- R7: MPN (none) -> RM06FTN1104; manf# RM06FTN1104 -> (none)
- U1: Config 3V3, 5V -> (none); MPN (none) -> MCP73831T-2ACI/OT; Variant (none) -> 3V3, 5V; manf# MCP73831T-2ACI/OT -> (none)
- U2: Config 3V3, 5V -> (none); MPN (none) -> TPS61090RSAR; Variant (none) -> 3V3, 5V; manf# TPS61090RSAR -> (none)
Changed lines of the file:
@@
 F 2 "Fuse:Fuse_0603_1608Metric" V 1180 1125 50  0001 C CNN
 F 3 "~" H 1250 1125 50  0001 C CNN
-F 4 "04000025WR" H 1250 1125 50  0001 C CNN "manf#"
+F 4 "04000025WR" H 1250 1125 50  0001 C CNN "MPN"
 F 5 "C135323" H 1250 1125 50  0001 C CNN "LCSC#"
 	1    1250 1125
@@
 F 2 "Resistor_SMD:R_0603_1608Metric" V 3930 2685 50  0001 C CNN
 F 3 "~" H 4000 2685 50  0001 C CNN
-F 4 "0603WAF3903T5E" H 4000 2685 50  0001 C CNN "manf#"
+F 4 "0603WAF3903T5E" H 4000 2685 50  0001 C CNN "MPN"
 F 5 "C23150" H 4000 2685 50  0001 C CNN "LCSC#"
 	1    4000 2685
@@
 F 2 "Resistor_SMD:R_0603_1608Metric" V 3930 3175 50  0001 C CNN
 F 3 "~" H 4000 3175 50  0001 C CNN
-F 4 "0603WAF3903T5E" H 4000 3175 50  0001 C CNN "manf#"
+F 4 "0603WAF3903T5E" H 4000 3175 50  0001 C CNN "MPN"
 F 5 "C23150" H 4000 3175 50  0001 C CNN "LCSC#"
 	1    4000 3175
@@
 F 2 "Diode_SMD:D_0603_1608Metric" H 1250 1635 50  0001 C CNN
 F 3 "~" H 1250 1635 50  0001 C CNN
-F 4 "3V3, 5V" H 1250 1635 50  0001 C CNN "Config"
+F 4 "3V3, 5V" H 1250 1635 50  0001 C CNN "Variant"
 	1    1250 1635
 	0    -1   -1   0
@@
 F 2 "Connector_JST:JST_PH_S2B-PH-SM4-TB_1x02-1MP_P2.00mm_Horizontal" H 3300 2875 50  0001 C CNN
 F 3 "~" H 3300 2875 50  0001 C CNN
-F 4 "" H 3300 2875 50  0001 C CNN "Config"
-F 5 "3V3, 5V" H 3300 2875 50  0001 C CNN "Config"
+F 4 "" H 3300 2875 50  0001 C CNN "Variant"
+F 5 "3V3, 5V" H 3300 2875 50  0001 C CNN "Variant"
 	1    3300 2875
 	-1   0    0    -1
@@
 F 2 "Capacitor_SMD:C_0603_1608Metric" H 1288 2275 50  0001 C CNN
 F 3 "~" H 1250 2425 50  0001 C CNN
-F 4 "CL10A106KP8NNNC" H 1250 2425 50  0001 C CNN "manf#"
+F 4 "CL10A106KP8NNNC" H 1250 2425 50  0001 C CNN "MPN"
 F 5 "C19702" H 1250 2425 50  0001 C CNN "LCSC#"
-F 6 "3V3, 5V" H 1250 2425 50  0001 C CNN "Config"
+F 6 "3V3, 5V" H 1250 2425 50  0001 C CNN "Variant"
 	1    1250 2425
 	1    0    0    -1
@@
 F 2 "Capacitor_SMD:C_0603_1608Metric" H 1788 2275 50  0001 C CNN
 F 3 "~" H 1750 2425 50  0001 C CNN
-F 4 "C0603C104M4RACTU" H 1750 2425 50  0001 C CNN "manf#"
+F 4 "C0603C104M4RACTU" H 1750 2425 50  0001 C CNN "MPN"
 F 5 "C14663" H 1750 2425 50  0001 C CNN "LCSC#"
-F 6 "3V3, 5V" H 1750 2425 50  0001 C CNN "Config"
+F 6 "3V3, 5V" H 1750 2425 50  0001 C CNN "Variant"
 	1    1750 2425
 	1    0    0    1
@@
 F 4 "" H 7500 2025 50  0001 C CNN "part#"
 F 5 "" H 7500 2025 50  0001 C CNN "LCSC"
-F 6 "744787068" H 7500 2025 50  0001 C CNN "manf#"
+F 6 "744787068" H 7500 2025 50  0001 C CNN "MPN"
 F 7 "C354631" H 7500 2025 50  0001 C CNN "LCSC#"
 	1    7500 2025
@@
 F 2 "Resistor_SMD:R_0603_1608Metric" V 2180 2900 50  0001 C CNN
 F 3 "~" H 2250 2900 50  0001 C CNN
-F 4 "0603WAF2001T5E" H 2250 2900 50  0001 C CNN "manf#"
+F 4 "0603WAF2001T5E" H 2250 2900 50  0001 C CNN "MPN"
 F 5 "C22975" H 2250 2900 50  0001 C CNN "LCSC#"
 	1    2250 2900
@@
 F 2 "Resistor_SMD:R_0603_1608Metric" V 6680 2175 50  0001 C CNN
 F 3 "~" H 6750 2175 50  0001 C CNN
-F 4 "0603WAF2003T5E" H 6750 2175 50  0001 C CNN "manf#"
+F 4 "0603WAF2003T5E" H 6750 2175 50  0001 C CNN "MPN"
 F 5 "C25811" H 6750 2175 50  0001 C CNN "LCSC#"
 	1    6750 2175
@@
 F 2 "Resistor_SMD:R_0603_1608Metric" V 7430 2525 50  0001 C CNN
 F 3 "~" H 7500 2525 50  0001 C CNN
-F 4 "WR06W2404FTL" H 7500 2525 50  0001 C CNN "manf#"
+F 4 "WR06W2404FTL" H 7500 2525 50  0001 C CNN "MPN"
 F 5 "C367738" H 7500 2525 50  0001 C CNN "LCSC#"
 	1    7500 2525
@@
 F 2 "Resistor_SMD:R_0603_1608Metric" V 7430 3025 50  0001 C CNN
 F 3 "~" H 7500 3025 50  0001 C CNN
-F 4 "0603WAF3903T5E" H 7500 3025 50  0001 C CNN "manf#"
+F 4 "0603WAF3903T5E" H 7500 3025 50  0001 C CNN "MPN"
 F 5 "C23150" H 7500 3025 50  0001 C CNN "LCSC#"
 	1    7500 3025
@@
 F 2 "Resistor_SMD:R_0603_1608Metric" V 9180 2225 50  0001 C CNN
 F 3 "~" H 9250 2225 50  0001 C CNN
-F 4 "RM06FTN1104" H 9250 2225 50  0001 C CNN "manf#"
+F 4 "RM06FTN1104" H 9250 2225 50  0001 C CNN "MPN"
 F 5 "C169875" H 9250 2225 50  0001 C CNN "LCSC#"
 	1    9250 2225
@@
 F 2 "Resistor_SMD:R_0603_1608Metric" V 9180 2775 50  0001 C CNN
 F 3 "~" H 9250 2775 50  0001 C CNN
-F 4 "0603WAF2003T5E" H 9250 2775 50  0001 C CNN "manf#"
+F 4 "0603WAF2003T5E" H 9250 2775 50  0001 C CNN "MPN"
 F 5 "C25811" H 9250 2775 50  0001 C CNN "LCSC#"
 	1    9250 2775
@@
 F 2 "Capacitor_SMD:C_0603_1608Metric" H 6038 2625 50  0001 C CNN
 F 3 "~" H 6000 2775 50  0001 C CNN
-F 4 "CL10A475KO8NNNC" H 6000 2775 50  0001 C CNN "manf#"
+F 4 "CL10A475KO8NNNC" H 6000 2775 50  0001 C CNN "MPN"
 F 5 "C19666" H 6000 2775 50  0001 C CNN "LCSC#"
 	1    6000 2775
@@
 F 2 "Capacitor_SMD:C_0603_1608Metric" H 6538 2625 50  0001 C CNN
 F 3 "~" H 6500 2775 50  0001 C CNN
-F 4 "CL10A106KP8NNNC" H 6500 2775 50  0001 C CNN "manf#"
+F 4 "CL10A106KP8NNNC" H 6500 2775 50  0001 C CNN "MPN"
 F 5 "C19702" H 6500 2775 50  0001 C CNN "LCSC#"
 	1    6500 2775
@@
 F 2 "Capacitor_SMD:C_0603_1608Metric" H 7038 2625 50  0001 C CNN
 F 3 "~" H 7000 2775 50  0001 C CNN
-F 4 "C0603C104M4RACTU" H 7000 2775 50  0001 C CNN "manf#"
+F 4 "C0603C104M4RACTU" H 7000 2775 50  0001 C CNN "MPN"
 F 5 "C14663" H 7000 2775 50  0001 C CNN "LCSC#"
 	1    7000 2775
@@
 F 2 "Capacitor_SMD:C_0603_1608Metric" H 9788 2375 50  0001 C CNN
 F 3 "~" H 9750 2525 50  0001 C CNN
-F 4 "C0603X105K9RACAUTO" H 9750 2525 50  0001 C CNN "manf#"
+F 4 "C0603X105K9RACAUTO" H 9750 2525 50  0001 C CNN "MPN"
 F 5 "C15849" H 9750 2525 50  0001 C CNN "LCSC#"
 	1    9750 2525
@@
 F 2 "Capacitor_SMD:C_0603_1608Metric" H 10288 2375 50  0001 C CNN
 F 3 "~" H 10250 2525 50  0001 C CNN
-F 4 "CL10A475KO8NNNC" H 10250 2525 50  0001 C CNN "manf#"
+F 4 "CL10A475KO8NNNC" H 10250 2525 50  0001 C CNN "MPN"
 F 5 "C19666" H 10250 2525 50  0001 C CNN "LCSC#"
 	1    10250 2525
@@
 F 2 "Package_TO_SOT_SMD:SOT-23-5" H 2800 2025 50  0001 L CIN
 F 3 "http://ww1.microchip.com/downloads/en/DeviceDoc/20001984g.pdf" H 2600 2225 50  0001 C CNN
-F 4 "MCP73831T-2ACI/OT " H 2750 2275 50  0001 C CNN "manf#"
+F 4 "MCP73831T-2ACI/OT " H 2750 2275 50  0001 C CNN "MPN"
 F 5 "C14879" H 2750 2275 50  0001 C CNN "LCSC#"
-F 6 "3V3, 5V" H 2750 2275 50  0001 C CNN "Config"
+F 6 "3V3, 5V" H 2750 2275 50  0001 C CNN "Variant"
 	1    2750 2275
 	1    0    0    -1
@@
 F 2 "Package_DFN_QFN:Texas_S-PVQFN-N16_EP2.7x2.7mm_ThermalVias" H 7550 1475 50  0001 L CNN
 F 3 "http://www.ti.com/lit/ds/symlink/tps61090.pdf" H 8650 1375 50  0001 L CNN
-F 4 "TPS61090RSAR" H 8500 2525 50  0001 C CNN "manf#"
+F 4 "TPS61090RSAR" H 8500 2525 50  0001 C CNN "MPN"
 F 5 "C206167" H 8500 2525 50  0001 C CNN "LCSC#"
-F 6 "3V3, 5V" H 8500 2525 50  0001 C CNN "Config"
+F 6 "3V3, 5V" H 8500 2525 50  0001 C CNN "Variant"
 	1    8500 2525
 	1    0    0    -1

Commit message: merged libs into one
Parts:
- A1: symbol ProMicro_BOOST-rescue:Sparkfun_Pro_Micro-MCU_Module -> ProMicro:Sparkfun_Pro_Micro
Changed lines of the file:
@@
 $EndComp
 $Comp
-L ProMicro_BOOST-rescue:Sparkfun_Pro_Micro-MCU_Module A1
+L ProMicro:Sparkfun_Pro_Micro A1
 U 1 1 5F84D072
 P 3500 5875

Commit message: BOOST_v1.8
Parts:
- A1: footprint Module:Sparkfun_Pro_Micro -> lib:ProMicro
- C1, C4: LCSC# C19702 -> (none)
- C2, C5: LCSC# C14663 -> (none); MPN C0603C104M4RACTU -> CL10B104KO8NNNC
- C3, C7: LCSC# C19666 -> (none)
- C6: LCSC# C15849 -> (none)
- F1: LCSC# C135323 -> (none)
- L1: LCSC# C354631 -> (none)
- R1, R2, R6: LCSC# C23150 -> (none)
- R3: LCSC# C22975 -> (none)
- R4, R8: LCSC# C25811 -> (none)
- R5: LCSC# C367738 -> (none)
- R7: LCSC# C169875 -> (none)
- U1: LCSC# C14879 -> (none)
- U2: LCSC# C206167 -> (none)
Connections:
- net LDO renamed LBO
Other:
- moved on the sheet: A1, C1, C2, C3, C4, C5, C6, C7, D1, F1, J1, JP1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
