File: CONN/ProMicro_CONN.sch (KiCad schematic (older format))
At the start: 20 parts, among them J1 AVR-JTAG-10, J2 UEXT_Host, J3 Display, SW1 reset, SW2 user

Commit message: dump
Parts:
- removed A1: Sparkfun_Pro_Micro_3V3, Module:Sparkfun_Pro_Micro, symbol MCU_Module:Sparkfun_Pro_Micro_3V3
- removed C1: 1µ, Capacitor_SMD:C_0603_1608Metric, symbol Device:C
- added A1: Sparkfun_Pro_Micro, Module:Sparkfun_Pro_Micro, symbol MCU_Module:Sparkfun_Pro_Micro
- LOGO1: footprint Symbol:OSHW-Logo2_7.3x6mm_SilkScreen -> Symbol:OSHW-Symbol_6.7x6mm_SilkScreen
Connections:
- net labels added: +5V, BTN, CIPO, COPI, CS1, RXD, SCK, SCL, SDA, TCK, TDI, TDO, TMS, TXD, ~RST
- net labels removed: A0, A1, A2, A3, D0, D1, D10, D14, D15, D16, D2, D3, D4, D5, D6, D7, D8, D9, Reset
- wire segments 76 -> 75
- no-connect marks 3 -> 6
Other:
- note removed: "BTN"
- note removed: "CS0"
- note removed: "CS1"
- note removed: "MISO"
- note removed: "MOSI"
- note removed: "RXD"
- note removed: "SCK"
- note removed: "SCL"
- note removed: "SDA"
- note removed: "TCK"
- note removed: "TDI"
- note removed: "TDO"
- note removed: "TMS"
- note removed: "TXD"
- note removed: "UEXT"
- note removed: "VBAT/2"

Commit message: clean
Parts:
- A1: symbol MCU_Module:Sparkfun_Pro_Micro -> ProMicro_CONN-rescue:Sparkfun_Pro_Micro-MCU_Module
Changed lines of the file:
@@
 SDA
 $Comp
-L MCU_Module:Sparkfun_Pro_Micro A1
+L ProMicro_CONN-rescue:Sparkfun_Pro_Micro-MCU_Module A1
 U 1 1 5F84D072
 P 9750 3000

Commit message: update schematic and PCBs
Parts:
- C2: MPN (none) -> CL10A105KB8NNNC; manf# CL10A105KB8NNNC -> (none)
- C3: MPN (none) -> CC0603KRX7R9BB104; manf# CC0603KRX7R9BB104 -> (none)
- D1: MPN (none) -> 19-217/GHC-YR1S2/3T; manf# 19-217/GHC-YR1S2/3T -> (none)
- R1, R2, R3, R4, R5, R6, R7, R9: MPN (none) -> 0603WAF4701T5E; manf# 0603WAF4701T5E -> (none)
- SW1, SW2: MPN (none) -> B3U-1000P; manf# B3U-1000P -> (none)
Changed lines of the file:
@@
 F 2 "Resistor_SMD:R_0603_1608Metric" V 3830 1500 50  0001 C CNN
 F 3 "~" H 3900 1500 50  0001 C CNN
-F 4 "0603WAF4701T5E" H 3900 1500 50  0001 C CNN "manf#"
+F 4 "0603WAF4701T5E" H 3900 1500 50  0001 C CNN "MPN"
 F 5 "C23162" H 3900 1500 50  0001 C CNN "LCSC#"
 	1    3900 1500
@@
 F 2 "Resistor_SMD:R_0603_1608Metric" V 4130 1500 50  0001 C CNN
 F 3 "~" H 4200 1500 50  0001 C CNN
-F 4 "0603WAF4701T5E" H 4200 1500 50  0001 C CNN "manf#"
+F 4 "0603WAF4701T5E" H 4200 1500 50  0001 C CNN "MPN"
 F 5 "C23162" H 4200 1500 50  0001 C CNN "LCSC#"
 	1    4200 1500
@@
 F 2 "Resistor_SMD:R_0603_1608Metric" V 4420 1500 50  0001 C CNN
 F 3 "~" H 4490 1500 50  0001 C CNN
-F 4 "0603WAF4701T5E" H 4490 1500 50  0001 C CNN "manf#"
+F 4 "0603WAF4701T5E" H 4490 1500 50  0001 C CNN "MPN"
 F 5 "C23162" H 4490 1500 50  0001 C CNN "LCSC#"
 	1    4490 1500
@@
 F 2 "Resistor_SMD:R_0603_1608Metric" V 4730 1500 50  0001 C CNN
 F 3 "~" H 4800 1500 50  0001 C CNN
-F 4 "0603WAF4701T5E" H 4800 1500 50  0001 C CNN "manf#"
+F 4 "0603WAF4701T5E" H 4800 1500 50  0001 C CNN "MPN"
 F 5 "C23162" H 4800 1500 50  0001 C CNN "LCSC#"
 	1    4800 1500
@@
 F 2 "Resistor_SMD:R_0603_1608Metric" V 6230 1500 50  0001 C CNN
 F 3 "~" H 6300 1500 50  0001 C CNN
-F 4 "0603WAF4701T5E" H 6300 1500 50  0001 C CNN "manf#"
+F 4 "0603WAF4701T5E" H 6300 1500 50  0001 C CNN "MPN"
 F 5 "C23162" H 6300 1500 50  0001 C CNN "LCSC#"
 	1    6300 1500
@@
 F 3 "~" H 9000 5500 50  0001 C CNN
 F 4 "C23162" H 9000 5500 50  0001 C CNN "LCSC#"
-F 5 "0603WAF4701T5E" H 9000 5500 50  0001 C CNN "manf#"
+F 5 "0603WAF4701T5E" H 9000 5500 50  0001 C CNN "MPN"
 	1    9000 5500
 	-1   0    0    1
@@
 F 3 "~" H 9500 5500 50  0001 C CNN
 F 4 "C23162" H 9500 5500 50  0001 C CNN "LCSC#"
-F 5 "0603WAF4701T5E" H 9500 5500 50  0001 C CNN "manf#"
+F 5 "0603WAF4701T5E" H 9500 5500 50  0001 C CNN "MPN"
 	1    9500 5500
 	-1   0    0    1
@@
 F 2 "LED_SMD:LED_0603_1608Metric" H 4800 2850 50  0001 C CNN
 F 3 "~" H 4800 2850 50  0001 C CNN
-F 4 "19-217/GHC-YR1S2/3T" H 4800 2850 50  0001 C CNN "manf#"
+F 4 "19-217/GHC-YR1S2/3T" H 4800 2850 50  0001 C CNN "MPN"
 F 5 "C72043" H 4800 2850 50  0001 C CNN "LCSC#"
 	1    4800 2850
@@
 F 2 "Capacitor_SMD:C_0603_1608Metric" H 6338 1850 50  0001 C CNN
 F 3 "~" H 6300 2000 50  0001 C CNN
-F 4 "CL10A105KB8NNNC" H 6300 2000 50  0001 C CNN "manf#"
+F 4 "CL10A105KB8NNNC" H 6300 2000 50  0001 C CNN "MPN"
 F 5 "C15849" H 6300 2000 50  0001 C CNN "LCSC#"
 	1    6300 2000
@@
 F 2 "Capacitor_SMD:C_0603_1608Metric" H 6478 5350 50  0001 C CNN
 F 3 "~" H 6440 5500 50  0001 C CNN
-F 4 "CC0603KRX7R9BB104" H 6440 5500 50  0001 C CNN "manf#"
+F 4 "CC0603KRX7R9BB104" H 6440 5500 50  0001 C CNN "MPN"
 F 5 "C14663" H 6440 5500 50  0001 C CNN "LCSC#"
 	1    6440 5500
@@
 F 2 "Button_Switch_SMD:SW_SPST_B3U-1000P" H 6000 2200 50  0001 C CNN
 F 3 "~" H 6000 2200 50  0001 C CNN
-F 4 " B3U-1000P" H 6000 2000 50  0001 C CNN "manf#"
+F 4 " B3U-1000P" H 6000 2000 50  0001 C CNN "MPN"
 	1    6000 2000
 	0    -1   -1   0
@@
 F 2 "Button_Switch_SMD:SW_SPST_B3U-1000P" H 7250 2200 50  0001 C CNN
 F 3 "~" H 7250 2200 50  0001 C CNN
-F 4 " B3U-1000P" H 7250 2000 50  0001 C CNN "manf#"
+F 4 " B3U-1000P" H 7250 2000 50  0001 C CNN "MPN"
 	1    7250 2000
 	0    -1   -1   0
@@
 F 2 "Resistor_SMD:R_0603_1608Metric" V 7180 1500 50  0001 C CNN
 F 3 "~" H 7250 1500 50  0001 C CNN
-F 4 "0603WAF4701T5E" H 7250 1500 50  0001 C CNN "manf#"
+F 4 "0603WAF4701T5E" H 7250 1500 50  0001 C CNN "MPN"
 F 5 "C23162" H 7250 1500 50  0001 C CNN "LCSC#"
 	1    7250 1500

Commit message: update PCBs to be stackable
Parts:
- A1: symbol ProMicro_CONN-rescue:Sparkfun_Pro_Micro-MCU_Module -> ProMicro:Sparkfun_Pro_Micro
Changed lines of the file:
@@
 SDA
 $Comp
-L ProMicro_CONN-rescue:Sparkfun_Pro_Micro-MCU_Module A1
+L ProMicro:Sparkfun_Pro_Micro A1
 U 1 1 5F84D072
 P 9750 3000

Commit message: CONN
Connections:
- wire segments 75 -> 74
Other:
- note added: "uses internal pull-up"
- moved on the sheet: R9
Changed lines of the file:
@@
 Sheet 1 1
 Title "ProMicro_CONN"
-Date "2020-07-11"
-Rev "v1.2"
+Date "2021-03-13"
+Rev "v1.3"
 Comp ""
 Comment1 ""
@@
 L Device:R R9
 U 1 1 5EB6D260
-P 7250 1500
-F 0 "R9" H 7350 1450 50  0000 L CNN
-F 1 "4k7" H 7350 1525 50  0000 L CNN
-F 2 "Resistor_SMD:R_0603_1608Metric" V 7180 1500 50  0001 C CNN
-F 3 "~" H 7250 1500 50  0001 C CNN
-F 4 "0603WAF4701T5E" H 7250 1500 50  0001 C CNN "MPN"
-F 5 "C23162" H 7250 1500 50  0001 C CNN "LCSC#"
-	1    7250 1500
-	-1   0    0    1
-$EndComp
-Wire Wire Line
-	7250 1650 7250 1700
-$Comp
-L power:+3V3 #PWR0124
-U 1 1 5EB6F14F
-P 7250 1200
-F 0 "#PWR0124" H 7250 1050 50  0001 C CNN
-F 1 "+3V3" H 7250 1350 50  0000 C CNN
-F 2 "" H 7250 1200 50  0001 C CNN
-F 3 "" H 7250 1200 50  0001 C CNN
-	1    7250 1200
-	1    0    0    -1
-$EndComp
-Wire Wire Line
-	7250 1200 7250 1350
-Connection ~ 7250 1700
+P 7250 2500
+F 0 "R9" H 7350 2450 50  0000 L CNN
+F 1 "4k7" H 7350 2525 50  0000 L CNN
+F 2 "Resistor_SMD:R_0603_1608Metric" V 7180 2500 50  0001 C CNN
+F 3 "~" H 7250 2500 50  0001 C CNN
+F 4 "0603WAF4701T5E" H 7250 2500 50  0001 C CNN "MPN"
+F 5 "C23162" H 7250 2500 50  0001 C CNN "LCSC#"
+	1    7250 2500
+	-1   0    0    1
+$EndComp
 Wire Wire Line
 	7250 1700 7250 1800
-Wire Wire Line
-	7250 2200 7250 2800
 $Comp
 L Connector:AVR-JTAG-10 J1
@@
 NoConn ~ 9250 3000
 NoConn ~ 9250 2300
+Wire Wire Line
+	7250 2800 7250 2650
+Wire Wire Line
+	7250 2350 7250 2200
+Text Notes 7250 1500 0    50   ~ 0
+uses internal pull-up
 $EndSCHEMATC
