File: _ANA/pcb/ANA.kicad_pcb (KiCad board)
At the start: 2 copper layers, 30.5 x 17.8 mm, 34 parts, among them J1 Conn_01x04, U1 TLV62569DDC, U2 MCP4725xxx-xCH, U3 TLV62569DDC, U4 MCP4725xxx-xCH, U5 INA260, U6 LTV-827S, U7 INA260

Commit message: cleanup using licenses
Routing:
- net +3V3: track 20.3 -> 23.8 mm
- net (no net): track 3.51 -> 0.00 mm
Other:
- net class Default removed
- net class Power removed
- net class small removed
- net class tiny removed
