File: _DEV/pcb/DEV.kicad_pcb (KiCad board)
At the start: 2 copper layers, 17.8 x 30.5 mm, 6 parts, among them J1 Conn_01x12, J2 Conn_01x12, J3 Conn_01x12, J4 Conn_01x12, J5 Conn_01x12

Commit message: cleanup using licenses
Connections:
- net ~RST renamed ~{RST}
Other:
- net class Default removed
- net class Power removed
- net class small removed
- net class tiny removed
