File: BOOST/pcb/BOOST.kicad_sch (KiCad schematic)
At the start: 25 parts, among them J1 JST, U1 MCP73831-2-OT, U2 TPS61090

Commit message: moved files
Parts:
- A1: footprint lib:ProMicro -> Module:Sparkfun_Pro_Micro
- U2: footprint Package_DFN_QFN:Texas_S-PVQFN-N16_EP2.7x2.7mm_ThermalVias -> Package_DFN_QFN:Texas_RSA_VQFN-16-1EP_4x4mm_P0.65mm_EP2.7x2.7mm_ThermalVias
Connections:
- net +3V3: now also A1.21 (VCC)
- net GND: now also A1.23 (GND), A1.3 (GND), A1.4 (GND)
- net STAT: now also A1.7 (D4/A6)
- net VBUS: now also A1.24 (RAW)

Commit message: update license
Other:
- company: nerdyscout -> Stefan Herold
- title: BOOST -> ProMicro_BOOST
Changed lines of the file:
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@@
 	(paper "A4")
 	(title_block
-		(title "BOOST")
-		(date "2021-04-05")
+		(title "ProMicro_BOOST")
+		(date "2025-01-05")
 		(rev "v1.5")
-		(company "nerdyscout")
+		(company "Stefan Herold")
+		(comment 1 "CERN-OHL-S-2.0")
 	)
 	(junction
@@
 		(at 273.05 173.99 0)
 		(unit 1)
-		(exclude_from_sim no)
+		(exclude_from_sim yes)
 		(in_bom yes)
 		(on_board yes)
@@
 			(at 273.05 173.99 0)
 			(effects
-				(font
-					(size 1.27 1.27)
-				)
-				(hide yes)
-			)
-		)
-		(property "Sim.Enable" "0"
-			(at 273.05 173.99 0)
-			(effects
