File: CONN/pcb/CONN.kicad_sch (KiCad schematic)
At the start: 20 parts, among them J1 AVR-JTAG-10, J2 UEXT_Host, J3 Display, SW1 reset, SW2 user, SW3 user

Commit message: update license
Other:
- company: nerdyscout -> Stefan Herold
Changed lines of the file:
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@@
 	(title_block
 		(title "CONN")
-		(date "2021-05-01")
+		(date "2025-01-05")
 		(rev "v1.4")
-		(company "nerdyscout")
+		(company "Stefan Herold")
+		(comment 1 "CERN-OHL-S-2.0")
 	)
 	(junction
@@
 		(at 274.32 175.26 0)
 		(unit 1)
-		(exclude_from_sim no)
+		(exclude_from_sim yes)
 		(in_bom yes)
 		(on_board yes)
@@
 			(at 274.32 175.26 0)
 			(effects
-				(font
-					(size 1.27 1.27)
-				)
-				(hide yes)
-			)
-		)
-		(property "Sim.Enable" "0"
-			(at 274.32 175.26 0)
-			(effects
