File: LOG/pcb/LOG.kicad_sch (KiCad schematic)
At the start: 16 parts, among them J1 Micro_SD_Card_Det, U1 DS3231MZ

Commit message: update license
Other:
- company: nerdyscout -> Stefan Herold
- title: LOG -> ProMicro_LOG
Changed lines of the file:
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@@
 	(paper "A4")
 	(title_block
-		(title "LOG")
+		(title "ProMicro_LOG")
 		(date "2020-10-12")
 		(rev "v1.2")
-		(company "nerdyscout")
+		(company "Stefan Herold")
+		(comment 1 "CERN-OHL-S-2.0")
 	)
 	(junction
@@
 		(at 274.32 175.26 0)
 		(unit 1)
-		(exclude_from_sim no)
+		(exclude_from_sim yes)
 		(in_bom yes)
 		(on_board yes)
@@
 			(at 274.32 175.26 0)
 			(effects
-				(font
-					(size 1.27 1.27)
-				)
-				(hide yes)
-			)
-		)
-		(property "Sim.Enable" "0"
-			(at 274.32 175.26 0)
-			(effects
