File: LORA/pcb/LORA.kicad_pcb (KiCad board)
At the start: 4 copper layers, 17.8 x 30.5 mm, 44 parts, among them J1 SMA, J2 COAX, U1 SX1276, U2 AS179-92LF, Y1 32Mhz

Commit message: update license
Other:
- board text added: "17,7800 mm x 30,4800 mm"
- board text removed: "30,4800 mm x 17,7800 mm"
