File: LORA/pcb/LORA.kicad_sch (KiCad schematic)
At the start: 44 parts, among them J1 SMA, J2 COAX, U1 SX1276, U2 AS179-92LF, Y1 32Mhz

Commit message: update license
Other:
- company: nerdyscout -> Stefan Herold
- title: LORA -> ProMicro_LORA
Changed lines of the file:
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@@
 	(paper "A4")
 	(title_block
-		(title "LORA")
-		(date "2024-12-26")
+		(title "ProMicro_LORA")
+		(date "2025-01-05")
 		(rev "v1.2")
-		(company "nerdyscout")
+		(company "Stefan Herold")
+		(comment 1 "CERN-OHL-S-2.0")
 	)
 	(junction
