File: POS/pcb/POS.kicad_sch (KiCad schematic)
At the start: 34 parts, among them J1 uFL, J2 Coax, U1 MPU-9250, U2 AP2112K-1.8, U3 SIM28ML

Commit message: update license
Other:
- company: (none) -> Stefan Herold
Changed lines of the file:
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@@
 	(title_block
 		(title "ProMicro_POS")
-		(date "2021-03-12")
+		(date "2025-01-05")
 		(rev "v3.4")
+		(company "Stefan Herold")
+		(comment 1 "CERN-OHL-S-2.0")
 	)
 	(junction
